Commit message: Imported upstream version '1.12.5' of 'upstream'

File: pal_pro_gripper_description/urdf/gripper.ros2_control.xacro (robot description, xacro)
@@ -23,5 +23,12 @@
       <command_interface name="position"/>
       <state_interface name="position">
-        <param name="initial_value">0.07938</param>
+        <!-- TODO: set initial_value back to 0.07938 when moving to Gazebo Harmonic or ROS 2 Jazzy -->
+        <!-- See https://robotics.stackexchange.com/questions/85506/how-to-do-mimic-joints-that-work-in-gazebo for more information -->
+        <xacro:if value="${gazebo_version == 'classic'}">
+          <param name="initial_value">0.07</param>
+        </xacro:if>
+        <xacro:if value="${gazebo_version == 'gazebo'}">
+          <param name="initial_value">0.0</param>
+        </xacro:if>
       </state_interface>
       <state_interface name="velocity"/>

File: pal_pro_gripper_description/urdf/gripper.urdf.xacro (robot description, xacro)
@@ -8,4 +8,12 @@
     </link>
     <xacro:property name="finger_joint_name" value="${name + '_finger_joint' if side == 'left' else name + '_finger_' + side + '_joint'}" />
+    <!-- TODO: set lower limit back to 0 when moving to Gazebo Harmonic or ROS 2 Jazzy -->
+    <!-- See https://github.com/gazebosim/gz-sim/issues/1684 for more information -->
+    <xacro:if value="${gazebo_version == 'classic'}">
+      <xacro:property name="gripper_lower_limit" value="0.0"/>
+    </xacro:if>
+    <xacro:if value="${gazebo_version == 'gazebo'}">
+      <xacro:property name="gripper_lower_limit" value="-1e-3"/>
+    </xacro:if>
     <joint name="${finger_joint_name}" type="prismatic">
       <xacro:origin_finger_joint reflect="${reflect}"/>
@@ -13,5 +21,6 @@
       <child link="${name}_screw_${side}_link"/>
       <axis xyz="0 1 0"/>
-      <limit lower="0.0" upper="0.07938" velocity="2" effort="0.1"/>
+      <limit lower="${gripper_lower_limit}" upper="0.07" velocity="2" effort="10.0"/>
+      <safety_controller k_position="20" k_velocity="20" soft_lower_limit="${gripper_lower_limit + gripper_eps}" soft_upper_limit="${0.07 - gripper_eps}" />
       <xacro:if value="${side == 'left'}">
         <dynamics damping="0.03"/>
@@ -132,4 +141,6 @@
     <xacro:property name="gripper_base_type" value="${'base_link_tc' if tool_changer else 'base_link_ntc'}" />
     <xacro:property name="finger_offset" value="${0.0 if tool_changer else 0.006}" />
+    <!--Constant parameters-->
+    <xacro:property name="gripper_eps" value="0.0" />
     <!-- Properties files -->
     <xacro:include filename="$(find pal_pro_gripper_description)/urdf/gripper.properties.xacro"/>
@@ -271,12 +282,14 @@
       <mu2>0.9</mu2>
     </gazebo>
-    <gazebo>
-      <plugin name="mimic_joint_plugin_right" filename="libgazebo_ros_mimic_joint.so">
-        <joint>gripper_finger_joint</joint>
-        <mimicJoint>gripper_finger_right_joint</mimicJoint>
-        <multiplier>1.0</multiplier>
-        <offset>0.0</offset>
-      </plugin>
-    </gazebo>
+    <xacro:if value="${gazebo_version == 'classic'}">
+      <gazebo>
+        <plugin name="mimic_joint_plugin_right" filename="libgazebo_ros_mimic_joint.so">
+          <joint>gripper_finger_joint</joint>
+          <mimicJoint>gripper_finger_right_joint</mimicJoint>
+          <multiplier>1.0</multiplier>
+          <offset>0.0</offset>
+        </plugin>
+      </gazebo>
+    </xacro:if>
     <!-- Base finger links -->
     <gazebo reference="${name}_base_finger_left_link">
