Commit message: Imported upstream version '1.11.3' of 'upstream'

File: pal_pro_gripper_description/robots/pal_pro_gripper.urdf.xacro (robot description, xacro)
@@ -13,9 +13,10 @@
     <!-- PROPERTIES -->
     <xacro:property name="tool_changer" value="$(arg tool_changer)" />
+    <xacro:property name="calibration_tool" value="$(arg calibration_tool)" />
     <xacro:property name="use_sim_time" value="$(arg use_sim_time)" />
     <xacro:property name="name" value="gripper"/>
     <!-- Mujoco properties -->
     <xacro:property name="sim_type" value="$(arg sim_type)" />
-    <xacro:property name="mj_control" value="${arg mj_control}"/>
+    <xacro:property name="mj_control" value="$(arg mj_control)"/>
     <xacro:property name="world_name" value="$(arg world_name)"/>
     <!-- INCLUDES -->
@@ -31,5 +32,5 @@
     <!-- ROBOT DEFINITION -->
     <link name="world"/>
-    <xacro:pal_pro_gripper tool_changer="${tool_changer}" name="${name}" parent="world">
+    <xacro:pal_pro_gripper tool_changer="${tool_changer}" name="${name}" parent="world" calibration_tool="${calibration_tool}">
         <origin xyz="0.0 0.0 0.08" rpy="0 0 0" />
     </xacro:pal_pro_gripper>

File: pal_pro_gripper_description/ros2_control/ros2_control.urdf.xacro (robot description, xacro)
@@ -30,5 +30,5 @@
       </hardware>
       <!-- pal-pro-gripper -->
-      <xacro:ros2_control_pal_pro_gripper name="gripper" reduction="1.0"  sim_type:="${sim_type}"/>
+      <xacro:ros2_control_pal_pro_gripper name="gripper" reduction="1.0"  sim_type="${sim_type}"/>
     </ros2_control>
   </xacro:macro>

File: pal_pro_gripper_description/urdf/gripper.properties.xacro (robot description, xacro)
@@ -25,5 +25,5 @@
     </xacro:macro>
     <xacro:macro name="origin_inner_finger_joint" params="reflect offset">
-        <origin xyz="0 ${reflect * 0.013977} ${0.078832 + offset}" rpy="1.5708 0.83776 ${reflect * 1.5708}" />
+        <origin xyz="-0.01482273272 0.00453176142 0.0" rpy="0.0 0.0 0.0" />
     </xacro:macro>
     <!-- Outer finger -->
@@ -36,5 +36,5 @@
     </xacro:macro>
     <xacro:macro name="origin_outer_finger_joint" params="reflect offset">
-        <origin xyz="0 ${reflect * 0.0288} ${0.0743 + offset}" rpy="1.5708 0.83776 ${reflect * 1.5708}" />
+        <origin xyz="0.0 ${reflect * 0.0288} 0.07565" rpy="1.5708 0 ${reflect * 1.5708}"/>
     </xacro:macro>
     <!-- Fingertip -->
@@ -47,5 +47,27 @@
     </xacro:macro>
     <xacro:macro name="origin_fingertip_joint" params="reflect">
-        <origin xyz="0 0.05 0" rpy="0 0 0.83776" />
+        <origin xyz="0 0.05 0" rpy="0 0 0" />
+    </xacro:macro>
+    <!-- Screw -->
+    <xacro:macro name="inertial_screw_link">
+        <inertial>
+            <origin xyz="0.0 0.0 0.0" rpy="0 0 0" />
+            <mass value="0.02" />
+            <inertia ixx="7.4666667e-07" ixy="0.0" ixz="0.0" iyy="7.4666667e-07" iyz="0.0" izz="1.6e-07" />
+        </inertial>
+    </xacro:macro>
+    <xacro:macro name="origin_finger_joint" params="reflect">
+        <origin xyz="-0.0178 0.0088 0.0" rpy="0 0 0"/>
+    </xacro:macro>
+    <!-- Base finger -->
+    <xacro:macro name="inertial_base_finger_link">
+        <inertial>
+            <origin xyz="0.0 0.0 0.0" rpy="0 0 0" />
+            <mass value="0.02" />
+            <inertia ixx="7.4666667e-07" ixy="0.0" ixz="0.0" iyy="7.4666667e-07" iyz="0.0" izz="1.6e-07" />
+        </inertial>
+    </xacro:macro>
+    <xacro:macro name="origin_base_finger_joint" params="reflect">
+    <origin xyz="0.0 ${reflect * 0.0288} 0.07565" rpy="1.5708 0 ${reflect * 1.5708}"/>
     </xacro:macro>
 </robot>

File: pal_pro_gripper_description/urdf/gripper.ros2_control.xacro (robot description, xacro)
@@ -23,14 +23,16 @@
       <command_interface name="position"/>
       <state_interface name="position">
-        <param name="initial_value">0.15</param>
+        <param name="initial_value">0.07938</param>
       </state_interface>
       <state_interface name="velocity"/>
       <state_interface name="effort"/>
     </joint>
-    <xacro:ros2_control_pal_pro_gripper_mimic_joint mimic_joint_name="${name}_outer_finger_right_joint" actuated_joint_name="${name}_finger_joint" multiplier="1"/>
-    <xacro:ros2_control_pal_pro_gripper_mimic_joint mimic_joint_name="${name}_inner_finger_right_joint" actuated_joint_name="${name}_finger_joint" multiplier="1"/>
-    <xacro:ros2_control_pal_pro_gripper_mimic_joint mimic_joint_name="${name}_fingertip_right_joint" actuated_joint_name="${name}_finger_joint" multiplier="-1"/>
-    <xacro:ros2_control_pal_pro_gripper_mimic_joint mimic_joint_name="${name}_inner_finger_left_joint" actuated_joint_name="${name}_finger_joint" multiplier="1"/>
-    <xacro:ros2_control_pal_pro_gripper_mimic_joint mimic_joint_name="${name}_fingertip_left_joint" actuated_joint_name="${name}_finger_joint" multiplier="-1"/>
+    <xacro:ros2_control_pal_pro_gripper_mimic_joint mimic_joint_name="${name}_outer_finger_right_joint" actuated_joint_name="${name}_finger_joint" multiplier="-8.28"/>
+    <xacro:ros2_control_pal_pro_gripper_mimic_joint mimic_joint_name="${name}_inner_finger_right_joint" actuated_joint_name="${name}_finger_joint" multiplier="-8.28"/>
+    <xacro:ros2_control_pal_pro_gripper_mimic_joint mimic_joint_name="${name}_fingertip_right_joint" actuated_joint_name="${name}_finger_joint" multiplier="8.28"/>
+    <xacro:ros2_control_pal_pro_gripper_mimic_joint mimic_joint_name="${name}_finger_right_joint" actuated_joint_name="${name}_finger_joint" multiplier="0.22"/>
+    <xacro:ros2_control_pal_pro_gripper_mimic_joint mimic_joint_name="${name}_outer_finger_left_joint" actuated_joint_name="${name}_finger_joint" multiplier="-8.28"/>
+    <xacro:ros2_control_pal_pro_gripper_mimic_joint mimic_joint_name="${name}_inner_finger_left_joint" actuated_joint_name="${name}_finger_joint" multiplier="-8.28"/>
+    <xacro:ros2_control_pal_pro_gripper_mimic_joint mimic_joint_name="${name}_fingertip_left_joint" actuated_joint_name="${name}_finger_joint" multiplier="8.28"/>
     <!-- Transmission only set to left finger joint, other joints are passive and mimic this
     joint-->

File: pal_pro_gripper_description/urdf/gripper.transmission.xacro (robot description, xacro)
@@ -15,8 +15,8 @@
   <xacro:macro name="pal_pro_gripper_transmission" params="name">
     <transmission name="${name}_trans">
-        <plugin>transmission_interface/SimpleTransmission</plugin>
+        <plugin>pal_pro_gripper_transmissions/PalGripperTransmission</plugin>
         <actuator name="${name}_actuator" role="actuator1"/>
         <joint name="${name}_joint" role="joint1">
-            <mechanical_reduction>1</mechanical_reduction>
+            <mechanical_reduction>0.001343799</mechanical_reduction>
         </joint>
     </transmission>

File: pal_pro_gripper_description/urdf/gripper.urdf.xacro (robot description, xacro)
@@ -3,64 +3,99 @@
   <!-- A finger of the pal_pro_gripper -->
   <xacro:macro name="pro_finger" params="name side reflect finger_offset:=0">
-    <!-- Inner finger -->
-    <link name="${name}_inner_finger_${side}_link">
-      <xacro:inertial_inner_finger_link />
-      <visual>
-        <origin xyz="0 0 0" rpy="0 0 0" />
-        <geometry>
-          <mesh filename="package://pal_pro_gripper_description/meshes/inner_finger.stl" />
-        </geometry>
-        <material name="">
-          <color rgba="0.752941176470588 0.752941176470588 0.752941176470588 1" />
-        </material>
-      </visual>
-      <collision>
-        <origin xyz="0 0 0" rpy="0 0 0" />
-        <geometry>
-          <mesh filename="package://pal_pro_gripper_description/meshes/inner_finger.stl" />
-        </geometry>
-      </collision>
-    </link>
-    <joint name="${name}_inner_finger_${side}_joint" type="revolute">
-      <xacro:origin_inner_finger_joint reflect="${reflect}" offset="${finger_offset}"/>
-      <parent link="${name}_base_link" />
-      <child link="${name}_inner_finger_${side}_link" />
-      <axis xyz="0 0 1" />
-      <limit lower="0" upper="${46 * deg_to_rad}" velocity="2" effort="0.1" />
-      <mimic joint="${name}_finger_joint" multiplier="1" offset="0" />
-    </joint>
-    <!-- Outer finger -->
-    <link name="${name}_outer_finger_${side}_link">
-      <xacro:inertial_outer_finger_link />
-      <visual>
-        <origin xyz="0 0 0" rpy="0 0 0" />
-        <geometry>
-          <mesh filename="package://pal_pro_gripper_description/meshes/outer_finger.stl" />
-        </geometry>
-        <material name="">
-          <color rgba="0.752941176470588 0.752941176470588 0.752941176470588 1" />
-        </material>
-      </visual>
-      <collision>
-        <origin xyz="0 0 0" rpy="0 0 0" />
-        <geometry>
-          <mesh filename="package://pal_pro_gripper_description/meshes/outer_finger.stl" />
-        </geometry>
-      </collision>
-    </link>
-    <!--  The left outer joint is set as gripper_finger_joint. All other joints are passive and will mimic this joint-->
-    <xacro:property name="outer_finger_joint_name" value="${name + '_finger_joint' if side == 'left' else name + '_outer_finger_' + side + '_joint'}" />
-    <joint name="${outer_finger_joint_name}" type="revolute">
-      <xacro:origin_outer_finger_joint reflect="${reflect}" offset="${finger_offset}"/>
-      <parent link="${name}_base_link" />
-      <child link="${name}_outer_finger_${side}_link" />
-      <axis xyz="0 0 1" />
-      <limit lower="0" upper="${54.431 * deg_to_rad}" velocity="2" effort="0.1" />
+    <!-- Screw link -->
+    <link name="${name}_screw_${side}_link">
+      <xacro:inertial_screw_link />
+    </link>
+    <xacro:property name="finger_joint_name" value="${name + '_finger_joint' if side == 'left' else name + '_finger_' + side + '_joint'}" />
+    <joint name="${finger_joint_name}" type="prismatic">
+      <xacro:origin_finger_joint reflect="${reflect}"/>
+      <parent link="${name}_base_finger_${side}_link"/>
+      <child link="${name}_screw_${side}_link"/>
+      <axis xyz="0 1 0"/>
+      <limit lower="0.0" upper="0.07938" velocity="2" effort="0.1"/>
       <xacro:if value="${side == 'left'}">
         <dynamics damping="0.03"/>
       </xacro:if>
       <xacro:unless value="${side == 'left'}">
-        <mimic joint="${name}_finger_joint" multiplier="1" offset="0" />
+        <mimic joint="${name}_finger_joint" multiplier="0.22" offset="0" />
       </xacro:unless>
+    </joint>
+    <!-- Gripper base finger link-->
+    <link name='${name}_base_finger_${side}_link'>
+      <xacro:inertial_base_finger_link/>
+      <visual>
+        <origin xyz="0 0 0" rpy="0 0 0"/>
+        <geometry>
+          <sphere radius="0.001"/>
+        </geometry>
+        <material name="">
+          <color rgba="0.752941176470588 0.752941176470588 0.752941176470588 1" />
+        </material>
+      </visual>
+      <collision>
+        <origin xyz="0 0 0" rpy="0 0 0"/>
+        <geometry>
+          <sphere radius="0.001"/>
+        </geometry>
+      </collision>
+    </link>
+    <joint name="${name}_base_finger_${side}_joint" type="fixed">
+      <xacro:origin_base_finger_joint reflect="${reflect}"/>
+      <parent link="${name}_base_link"/>
+      <child link="${name}_base_finger_${side}_link"/>
+    </joint>
+    <!-- Inner finger -->
+    <link name="${name}_inner_finger_${side}_link">
+      <xacro:inertial_inner_finger_link />
+      <visual>
+        <origin xyz="0 0 0" rpy="0 0 0"/>
+        <geometry>
+          <mesh filename="package://pal_pro_gripper_description/meshes/inner_finger.stl"/>
+        </geometry>
+        <material name="">
+          <color rgba="0.752941176470588 0.752941176470588 0.752941176470588 1" />
+        </material>
+      </visual>
+      <collision>
+        <origin xyz="0 0 0" rpy="0 0 0"/>
+        <geometry>
+          <mesh filename="package://pal_pro_gripper_description/meshes/inner_finger.stl"/>
+        </geometry>
+      </collision>
+    </link>
+    <joint name="${name}_inner_finger_${side}_joint" type="revolute">
+      <xacro:origin_inner_finger_joint reflect="${reflect}" offset="${finger_offset}"/>
+      <parent link="${name}_base_finger_${side}_link"/>
+      <child link="${name}_inner_finger_${side}_link"/>
+      <axis xyz="0 0 1"/>
+      <limit lower="${-42.840* deg_to_rad}" upper="${8.001 * deg_to_rad}" velocity="2" effort="0.1"/>
+      <mimic joint="${name}_finger_joint" multiplier="-8.28" offset="0.0"/>
+    </joint>
+    <!-- Outer finger -->
+    <link name="${name}_outer_finger_${side}_link">
+      <xacro:inertial_outer_finger_link />
+      <visual>
+        <origin xyz="0 0 0" rpy="0 0 0"/>
+        <geometry>
+          <mesh filename="package://pal_pro_gripper_description/meshes/outer_finger.stl"/>
+        </geometry>
+        <material name="">
+          <color rgba="0.752941176470588 0.752941176470588 0.752941176470588 1" />
+        </material>
+      </visual>
+      <collision>
+        <origin xyz="0 0 0" rpy="0 0 0"/>
+        <geometry>
+          <mesh filename="package://pal_pro_gripper_description/meshes/outer_finger.stl"/>
+        </geometry>
+      </collision>
+    </link>
+    <joint name="${name}_outer_finger_${side}_joint" type="revolute">
+      <xacro:origin_outer_finger_joint reflect="${reflect}" offset="${finger_offset}"/>
+      <parent link="${name}_base_link"/>
+      <child link="${name}_outer_finger_${side}_link"/>
+      <axis xyz="0 0 1"/>
+      <limit lower="${-42.840 * deg_to_rad}" upper="${8.001 * deg_to_rad}" velocity="2" effort="0.1"/>
+      <mimic joint="${name}_finger_joint" multiplier="-8.28" offset="0.0"/>
     </joint>
     <!-- Fingertip -->
@@ -68,30 +103,30 @@
       <xacro:inertial_fingertip_link />
       <visual>
-        <origin xyz="0 0 0" rpy="0 0 0" />
-        <geometry>
-          <mesh filename="package://pal_pro_gripper_description/meshes/fingertip.stl" />
-        </geometry>
-        <material name="">
-          <color rgba="0.752941176470588 0.752941176470588 0.752941176470588 1" />
-        </material>
-      </visual>
-      <collision>
-        <origin xyz="0 0 0" rpy="0 0 0" />
-        <geometry>
-          <mesh filename="package://pal_pro_gripper_description/meshes/fingertip.stl" />
+        <origin xyz="0 0 0" rpy="0 0 0"/>
+        <geometry>
+          <mesh filename="package://pal_pro_gripper_description/meshes/fingertip.stl"/>
+        </geometry>
+        <material name="">
+          <color rgba="0.752941176470588 0.752941176470588 0.752941176470588 1" />
+        </material>
+      </visual>
+      <collision>
+        <origin xyz="0 0 0" rpy="0 0 0"/>
+        <geometry>
+          <mesh filename="package://pal_pro_gripper_description/meshes/fingertip.stl"/>
         </geometry>
       </collision>
     </link>
     <joint name="${name}_fingertip_${side}_joint" type="revolute">
-      <xacro:origin_fingertip_joint reflect="${reflect}" />
-      <parent link="${name}_inner_finger_${side}_link" />
-      <child link="${name}_fingertip_${side}_link" />
-      <axis xyz="0 0 1" />
-      <limit lower="${-46 * deg_to_rad}" upper="0" velocity="2" effort="0.1" />
-      <mimic joint="${name}_finger_joint" multiplier="-1" offset="0" />
+      <xacro:origin_fingertip_joint reflect="${reflect}"/>
+      <parent link="${name}_inner_finger_${side}_link"/>
+      <child link="${name}_fingertip_${side}_link"/>
+      <axis xyz="0 0 1"/>
+      <limit lower="${-8.001 * deg_to_rad}" upper="${42.840 * deg_to_rad}" velocity="2" effort="0.1"/>
+      <mimic joint="${name}_finger_joint" multiplier="8.28" offset="0.0"/>
     </joint>
   </xacro:macro>
   <!-- GRIPPER DEFINITION -->
-  <xacro:macro name="pal_pro_gripper" params="tool_changer:=False name parent *origin">
+  <xacro:macro name="pal_pro_gripper" params="tool_changer:=False name parent *origin calibration_tool:=False">
     <!-- Vesion name depending if it is a prototype -->
     <xacro:property name="gripper_base_type" value="${'base_link_tc' if tool_changer else 'base_link_ntc'}" />
@@ -128,15 +163,51 @@
     </joint>
     <!-- Grasping Frame -->
-    <joint name="${name}_grasping_frame_joint" type="fixed">
-      <parent link="${name}_base_link"/>
-      <child link="${name}_grasping_link"/>
-      <origin xyz="0.0 0 0.157157" rpy="0 -1.57 0" />
-    </joint>
-    <link name="${name}_grasping_link">
-      <inertial>
-        <mass value="1e-9" />
-        <inertia ixx="1e-9" ixy="0.0" ixz="0.0" iyy="1e-9" iyz="0.0" izz="1e-9" />
-      </inertial>
-    </link>
+    <!-- If calibration tool is used, add the visible tool to end effector to avoid collisions -->
+    <xacro:if value="${calibration_tool}">
+      <joint name="${name}_grasping_frame_joint" type="fixed">
+        <parent link="${name}_base_link"/>
+        <child link="${name}_grasping_link"/>
+        <origin xyz="0.0 0.0 0.13" rpy="0 0 0" />
+      </joint>
+      <link name="${name}_grasping_link">
+        <inertial>
+          <mass value="0.1" />
+          <origin xyz="0 0 0.1" rpy="0 0 0" />
+          <inertia ixx="0.000341" ixy="0" ixz="0" iyy="0.000241" iyz="0" izz="0.000101" />
+        </inertial>
+        <visual>
+          <origin xyz="0 0 0.1" rpy="0 0 0" />
+          <geometry>
+            <box size="0.01 0.12 0.09" />
+          </geometry>
+          <material name="grasp_box_color">
+            <color rgba="0 0 1 1" />
+          </material>
+        </visual>
+        <collision>
+          <origin xyz="0 0 0.1" rpy="0 0 0" />
+          <geometry>
+            <box size="0.01 0.12 0.09" />
+          </geometry>
+        </collision>
+      </link>
+    </xacro:if>
+    <gazebo reference="${name}_grasping_link">
+        <material>Gazebo/Blue</material>
+        <turnGravityOff>true</turnGravityOff>
+      </gazebo>
+    <xacro:unless value="${calibration_tool}">
+      <joint name="${name}_grasping_frame_joint" type="fixed">
+        <parent link="${name}_base_link"/>
+        <child link="${name}_grasping_link"/>
+        <origin xyz="0.0 0.0 0.157157" rpy="0 -1.57 0" />
+      </joint>
+      <link name="${name}_grasping_link">
+        <inertial>
+          <mass value="1e-9" />
+          <inertia ixx="1e-9" ixy="0.0" ixz="0.0" iyy="1e-9" iyz="0.0" izz="1e-9" />
+        </inertial>
+      </link>
+    </xacro:unless>
     <!-- Fingers -->
     <xacro:pro_finger name="${name}" side="left" reflect="-1" finger_offset="${finger_offset}"/>
@@ -178,11 +249,44 @@
       <mu2>0.9</mu2>
     </gazebo>
+    <!-- Screw links -->
     <gazebo reference="${name}_finger_joint">
-      <implicitSpringDamper>1</implicitSpringDamper>
-      <provideFeedback>1</provideFeedback>
+      <material>Gazebo/DarkGrey</material>
+      <mu1>0.9</mu1>
+      <mu2>0.9</mu2>
     </gazebo>
     <gazebo reference="${name}_finger_joint">
-      <implicitSpringDamper>1</implicitSpringDamper>
-      <provideFeedback>1</provideFeedback>
+      <material>Gazebo/DarkGrey</material>
+      <mu1>0.9</mu1>
+      <mu2>0.9</mu2>
+    </gazebo>
+    <!-- Base finger links -->
+    <gazebo reference="${name}_base_finger_left_link">
+      <material>Gazebo/DarkGrey</material>
+      <mu1>0.9</mu1>
+      <mu2>0.9</mu2>
+    </gazebo>
+    <gazebo reference="${name}_base_finger_right_link">
+      <material>Gazebo/DarkGrey</material>
+      <mu1>0.9</mu1>
+      <mu2>0.9</mu2>
+    </gazebo>
+    <gazebo>
+      <plugin name="mimic_joint_plugin_right" filename="libgazebo_ros_mimic_joint.so">
+        <joint>gripper_finger_joint</joint>
+        <mimicJoint>gripper_finger_right_joint</mimicJoint>
+        <multiplier>1.0</multiplier>
+        <offset>0.0</offset>
+      </plugin>
+    </gazebo>
+    <!-- Base finger links -->
+    <gazebo reference="${name}_base_finger_left_link">
+      <material>Gazebo/DarkGrey</material>
+      <mu1>0.9</mu1>
+      <mu2>0.9</mu2>
+    </gazebo>
+    <gazebo reference="${name}_base_finger_right_link">
+      <material>Gazebo/DarkGrey</material>
+      <mu1>0.9</mu1>
+      <mu2>0.9</mu2>
     </gazebo>
   </xacro:macro>
